File: Hardware/nrf_rgb_clock.kicad_sch (KiCad schematic)
At the start: 16 parts, among them U1 NRF54L15-CAAA-Rx, Y2 32MHz

Commit message: initial commit
Parts:
- added U2, U3: ~, LED_SMD:LED_WS2812_PLCC6_5.0x5.0mm_P1.6mm, symbol ProjectSymbols:WS2813B-5V
Connections:
- net GND: now also U2.5 (GND), U3.5 (GND)
- new net: U2.1 (BO), U3.6 (BI)
- new net: U2.3 (DO), U3.4 (DI)
- new net +5V: U2.2 (VCC), U3.2 (VCC)
Other:
- note added: "7 segments per LED x 4 + 2 for dots + 1 for circular display: 31 segments nrf has 31 GPIOs in QFN48 package, 32 GPIOs in WLCSP package"

Commit message: led placement on pcb
Parts:
- removed U2, U3: ~, LED_SMD:LED_WS2812_PLCC6_5.0x5.0mm_P1.6mm, symbol ProjectSymbols:WS2813B-5V
- added D116, D117: ~, LED_SMD:LED_WS2812_PLCC6_5.0x5.0mm_P1.6mm, symbol ProjectSymbols:WS2813B-5V
- added H1, H2, H3, H4: MountingHole, MountingHole:MountingHole_3.2mm_M3, symbol Mechanical:MountingHole
- renumbered C2 to C1, C1 to C2, C6 to C4, C7 to C5, C8 to C6, C9 to C7, C5 to C8, C4 to C9, L4 to L1, L1 to L2, L2 to L3, L3 to L4, Y2 to Y1
Connections:
- net +5V: now also D116.2 (VCC), D117.2 (VCC)
- net GND: now also D116.5 (GND), D117.5 (GND)
- new net: D116.3 (DO), D117.4 (DI)
- new net: D116.1 (BO), D117.6 (BI)
- new net led_segment1/LED_BO: D116.4 (DI)
- new net led_segment1/LED_DO: D116.6 (BI)
- new net led_segment2/LED_BI: D117.1 (BO)
- new net led_segment2/LED_DI: D117.3 (DO)
Other:
- added sheet led_circle (led_circle.kicad_sch)
- added sheet led_segment (led_segment.kicad_sch)
- added sheet led_segment1 (led_segment.kicad_sch)
- added sheet led_segment2 (led_segment.kicad_sch)
- added sheet led_segment3 (led_segment.kicad_sch)
- note added: "nrf has 31 GPIOs in QFN48 package, 32 GPIOs in WLCSP package divide display in to 7 segment and circular array. Use only 2 pins"
- note removed: "7 segments per LED x 4 + 2 for dots + 1 for circular display: 31 segments nrf has 31 GPIOs in QFN48 package, 32 GPIOs in WLCSP package"

Commit message: Added bitoffsets and antenna
Parts:
- added AE1: 2450AT43A100E, ProjectFootprints:2450AT43A100E, symbol Device:Antenna_Chip
- Y1: footprint (none) -> Crystal:Crystal_SMD_3225-4Pin_3.2x2.5mm; LCSC (none) -> C37635386
Connections:
- net NRF_RF: no longer L2.2
- net LED_CIRCLE: now reaches U1.B4 (P1.13)
- net LED_SEGMENTS: now reaches U1.B5 (P1.14)
- net NRF_XC_OPT1: no longer names the net of U1.C5 (P1.00)
- net NRF_XC_OPT2: no longer names the net of U1.C6 (P1.01)
- new net: AE1.1 (FEED), L2.2
- no-connect marks 0 -> 5
Other:
- note added: "A"
- note added: "A_0 = 0; 0 B_0 = 96; 12 C_0 = 192; 24 D_0 = 288; 36 E_0 = 384; 48 F_0 = 480; 60 G_0 = 576; 72"
- note added: "B"
- note added: "C"
- note added: "D"
- note added: "E"
- note added: "F"
- note added: "G"
- note added: "Horizontal mount if possible for better gain and efficiency"
- note added: "LED"
- note added: "P1"
- note added: "P2"
- note added: "bit_offset = 0; byte_offset = 0"
- note added: "bit_offset = 1344; byte_offset = 168 segments: P1_0: 0 P2_0: 24"
- note added: "bit_offset = 1392; byte_offset = 172"
- note added: "bit_offset = 2064; byte_offset = 258"
- note added: "bit_offset = 672; byte_offset = 84"
- moved on the sheet: C1, C2, C3, C4, C5, C6, C7, C8, C9, D116, D117, FB1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

Commit message: added LCSC number and datasheets
Parts:
- C1: footprint (none) -> Capacitor_SMD:C_0805_2012Metric; LCSC (none) -> C2932476
- C2, C3: footprint Capacitor_SMD:C_0201_0603Metric -> Capacitor_SMD:C_0402_1005Metric; LCSC (none) -> C1581
- C4, C5: value 2u2 -> 2u2 50V; footprint Capacitor_SMD:C_0201_0603Metric -> Capacitor_SMD:C_0603_1608Metric; LCSC (none) -> C7432769
- C6: value 10n -> 10n 50V; LCSC (none) -> C5142551
- C7: value 3p9 -> 3p9 50V; LCSC (none) -> C22374845
- C8, C9: value 1p2 -> 1p2 50V; LCSC (none) -> C22374839
- D116, D117: value ~ -> WS2813b
- FB1: footprint (none) -> Resistor_SMD:R_0402_1005Metric; LCSC (none) -> C337874
- L1: footprint LED_SMD:LED_0402_1005Metric -> LED_SMD:LED_0201_0603Metric
- L2: footprint Inductor_SMD:L_0201_0603Metric -> LED_SMD:LED_0201_0603Metric
Changed lines of the file:
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@@
 			)
 		)
-		(property "Value" "3p9"
+		(property "Value" "3p9 50V"
 			(at 119.38 135.8835 0)
 			(effects
@@
 			)
 		)
-		(property "Datasheet" "~"
+		(property "Datasheet" "https://www.lcsc.com/datasheet/lcsc_datasheet_2404101552_HRE-CGA0201C0G3R9C500ET_C22374845.pdf"
 			(at 121.92 134.62 0)
 			(effects
@@
 		)
 		(property "Description" "Unpolarized capacitor, small symbol"
+			(at 121.92 134.62 0)
+			(effects
+				(font
+					(size 1.27 1.27)
+				)
+				(hide yes)
+			)
+		)
+		(property "LCSC" "C22374845"
 			(at 121.92 134.62 0)
 			(effects
@@
 			)
 		)
-		(property "Value" "~"
+		(property "Value" "WS2813b"
 			(at 301.9141 50.8 0)
 			(effects
@@
 			)
 		)
-		(property "Footprint" ""
+		(property "Footprint" "Capacitor_SMD:C_0805_2012Metric"
 			(at 124.46 39.37 0)
 			(effects
@@
 			)
 		)
-		(property "Datasheet" "~"
+		(property "Datasheet" "https://www.lcsc.com/datasheet/lcsc_datasheet_2201121530_Samsung-Electro-Mechanics-CL21A106KBYQNNE_C2932476.pdf"
 			(at 124.46 39.37 0)
 			(effects
@@
 		)
 		(property "Description" "Unpolarized capacitor, small symbol"
+			(at 124.46 39.37 0)
+			(effects
+				(font
+					(size 1.27 1.27)
+				)
+				(hide yes)
+			)
+		)
+		(property "LCSC" "C2932476"
 			(at 124.46 39.37 0)
 			(effects
@@
 			)
 		)
-		(property "Value" "2u2"
+		(property "Value" "2u2 50V"
 			(at 92.71 123.1835 0)
 			(effects
@@
 			)
 		)
-		(property "Footprint" "Capacitor_SMD:C_0201_0603Metric"
+		(property "Footprint" "Capacitor_SMD:C_0603_1608Metric"
 			(at 95.25 121.92 0)
 			(effects
@@
 			)
 		)
-		(property "Datasheet" "~"
+		(property "Datasheet" "https://www.lcsc.com/datasheet/lcsc_datasheet_2411041754_Chinocera-HGC0603R5225K500NTHJ_C7432769.pdf"
 			(at 95.25 121.92 0)
 			(effects
@@
 		)
 		(property "Description" "Unpolarized capacitor, small symbol"
+			(at 95.25 121.92 0)
+			(effects
+				(font
+					(size 1.27 1.27)
+				)
+				(hide yes)
+			)
+		)
+		(property "LCSC" "C7432769"
 			(at 95.25 121.92 0)
 			(effects
@@
 			)
 		)
-		(property "Value" "2u2"
+		(property "Value" "2u2 50V"
 			(at 101.6 135.8835 0)
 			(effects
@@
 			)
 		)
-		(property "Footprint" "Capacitor_SMD:C_0201_0603Metric"
+		(property "Footprint" "Capacitor_SMD:C_0603_1608Metric"
 			(at 104.14 134.62 0)
 			(effects
@@
 			)
 		)
-		(property "Datasheet" "~"
+		(property "Datasheet" "https://www.lcsc.com/datasheet/lcsc_datasheet_2411041754_Chinocera-HGC0603R5225K500NTHJ_C7432769.pdf"
 			(at 104.14 134.62 0)
 			(effects
@@
 			)
 		)
+		(property "LCSC" "C7432769"
+			(at 104.14 134.62 0)
+			(effects
+				(font
+					(size 1.27 1.27)
+				)
+				(hide yes)
+			)
+		)
 		(pin "2"
 		)
@@
 			)
 		)
-		(property "Footprint" "Inductor_SMD:L_0201_0603Metric"
+		(property "Footprint" "LED_SMD:LED_0201_0603Metric"
 			(at 168.91 177.8 0)
 			(effects
@@
 			)
 		)
-		(property "Datasheet" "~"
+		(property "Datasheet" ""
 			(at 168.91 177.8 0)
 			(effects
@@
 		)
 		(property "Description" "Inductor, small symbol"
+			(at 168.91 177.8 0)
+			(effects
+				(font
+					(size 1.27 1.27)
+				)
+				(hide yes)
+			)
+		)
+		(property "LCSC" ""
 			(at 168.91 177.8 0)
 			(effects
@@
 			)
 		)
-		(property "Value" "10n"
+		(property "Value" "10n 50V"
 			(at 110.49 135.8835 0)
 			(effects
@@
 			)
 		)
-		(property "Datasheet" "~"
+		(property "Datasheet" "https://www.lcsc.com/datasheet/lcsc_datasheet_2209011730_CCTC-TCC0201X7R103K500ZT_C5142551.pdf"
 			(at 113.03 134.62 0)
 			(effects
@@
 			)
 		)
+		(property "LCSC" "C5142551"
+			(at 113.03 134.62 0)
+			(effects
+				(font
+					(size 1.27 1.27)
+				)
+				(hide yes)
+			)
+		)
 		(pin "2"
 		)
@@
 			)
 		)
-		(property "Value" "1p2"
+		(property "Value" "1p2 50V"
 			(at 166.37 184.1435 0)
 			(effects
@@
 			)
 		)
-		(property "Datasheet" "~"
+		(property "Datasheet" "https://www.lcsc.com/datasheet/lcsc_datasheet_2404101552_HRE-CGA0201C0G1R2C500ET_C22374839.pdf"
 			(at 163.83 182.88 0)
 			(effects
@@
 		)
 		(property "Description" "Unpolarized capacitor, small symbol"
+			(at 163.83 182.88 0)
+			(effects
+				(font
+					(size 1.27 1.27)
+				)
+				(hide yes)
+			)
+		)
+		(property "LCSC" "C22374839"
 			(at 163.83 182.88 0)
 			(effects
@@
 			)
 		)
-		(property "Footprint" "Capacitor_SMD:C_0201_0603Metric"
+		(property "Footprint" "Capacitor_SMD:C_0402_1005Metric"
 			(at 153.67 39.37 0)
 			(effects
@@
 			)
 		)
-		(property "Datasheet" "~"
+		(property "Datasheet" "https://www.lcsc.com/datasheet/lcsc_datasheet_2304140030_FH--Guangdong-Fenghua-Advanced-Tech-0402F104M500NT_C1581.pdf"
 			(at 153.67 39.37 0)
 			(effects
@@
 			)
 		)
+		(property "LCSC" "C1581"
+			(at 153.67 39.37 0)
+			(effects
+				(font
+					(size 1.27 1.27)
+				)
+				(hide yes)
+			)
+		)
 		(pin "2"
 		)
@@
 			)
 		)
-		(property "Footprint" ""
+		(property "Footprint" "Resistor_SMD:R_0402_1005Metric"
 			(at 102.362 121.92 90)
 			(effects
@@
 			)
 		)
-		(property "Datasheet" "~"
+		(property "Datasheet" "https://www.lcsc.com/datasheet/lcsc_datasheet_2304140030_Murata-Electronics-BLM15BD121SN1D_C337874.pdf"
 			(at 104.14 121.92 0)
 			(effects
@@
 			)
 		)
+		(property "LCSC" "C337874"
+			(at 104.14 121.92 0)
+			(effects
+				(font
+					(size 1.27 1.27)
+				)
+				(hide yes)
+			)
+		)
 		(pin "2"
 		)
@@
 			)
 		)
-		(property "Value" "~"
+		(property "Value" "WS2813b"
 			(at 280.3241 50.8 0)
 			(effects
@@
 			)
 		)
-		(property "Value" "1p2"
+		(property "Value" "1p2 50V"
 			(at 156.21 184.1435 0)
 			(effects
@@
 			)
 		)
-		(property "Datasheet" "~"
+		(property "Datasheet" "https://www.lcsc.com/datasheet/lcsc_datasheet_2404101552_HRE-CGA0201C0G1R2C500ET_C22374839.pdf"
 			(at 153.67 182.88 0)
 			(effects
@@
 		)
 		(property "Description" "Unpolarized capacitor, small symbol"
+			(at 153.67 182.88 0)
+			(effects
+				(font
+					(size 1.27 1.27)
+				)
+				(hide yes)
+			)
+		)
+		(property "LCSC" "C22374839"
 			(at 153.67 182.88 0)
 			(effects
@@
 			)
 		)
-		(property "Footprint" "LED_SMD:LED_0402_1005Metric"
+		(property "Footprint" "LED_SMD:LED_0201_0603Metric"
 			(at 104.14 111.76 0)
 			(effects
@@
 			)
 		)
-		(property "Datasheet" "~"
+		(property "Datasheet" ""
 			(at 104.14 111.76 0)
 			(effects
@@
 		)
 		(property "Description" "Inductor, small symbol"
+			(at 104.14 111.76 0)
+			(effects
+				(font
+					(size 1.27 1.27)
+				)
+				(hide yes)
+			)
+		)
+		(property "LCSC" ""
 			(at 104.14 111.76 0)
 			(effects
@@
 			)
 		)
-		(property "Footprint" "Capacitor_SMD:C_0201_0603Metric"
+		(property "Footprint" "Capacitor_SMD:C_0402_1005Metric"
 			(at 137.16 39.37 0)
 			(effects
@@
 			)
 		)
-		(property "Datasheet" "~"
+		(property "Datasheet" "https://www.lcsc.com/datasheet/lcsc_datasheet_2304140030_FH--Guangdong-Fenghua-Advanced-Tech-0402F104M500NT_C1581.pdf"
 			(at 137.16 39.37 0)
 			(effects
@@
 			(at 137.16 39.37 0)
 			(effects
+				(font
+					(size 1.27 1.27)
+				)
+				(hide yes)
+			)
+		)
+		(property "LCSC" "C1581"
+			(at 137.16 39.37 0)
+			(effects

Commit message: progressed layout
Parts:
- added C10, C11: 4u7 100VDC, Capacitor_SMD:C_1206_3216Metric, symbol Device:C_Small
- added C12: 100n 100VDC, Capacitor_SMD:C_0805_2012Metric, symbol Device:C_Small
- added C13, C14: 22u 6.3V, Capacitor_SMD:C_0805_2012Metric, symbol Device:C_Small
- added C15: 15p, Capacitor_SMD:C_0805_2012Metric, symbol Device:C_Small
- added C16: 22n, Capacitor_SMD:C_0805_2012Metric, symbol Device:C_Small
- added C17, C18: ?p, Capacitor_SMD:C_0201_0603Metric, symbol Device:C_Small
- added D174: ACDBMS2100-HF, Diode_SMD:D_SOD-123F, symbol Device:D_Schottky_Small_Filled
- added J1: Conn_01x02, ProjectFootprints:SHDR4W113P700X508_2X2_1039X1200X1200P, symbol Connector_Generic:Conn_01x02
- added L5: 10u, ProjectFootprints:NRS5040T3R3NMGJV, symbol Device:L_Small
- added R1: 0R, Resistor_SMD:R_0805_2012Metric, symbol Device:R_Small
- added R2: 210k, Resistor_SMD:R_0805_2012Metric, symbol Device:R_Small
- added R3: 68k, Resistor_SMD:R_0805_2012Metric, symbol Device:R_Small
- added R4: 47k, Resistor_SMD:R_0805_2012Metric, symbol Device:R_Small
- added TP1, TP2: TestPoint, TestPoint:TestPoint_THTPad_2.0x2.0mm_Drill1.0mm, symbol Connector:TestPoint
- added U2: MP4562, ProjectFootprints:MP4562, symbol ProjectSymbols:MP4562
Connections:
- net GND: now also C10.2, C11.2, C13.2, C14.2, C16.2, C17.2, C18.2, D174.2 (A), J1.2 (Pin_2), R3.2, R4.2, TP2.1, U2.2 (GND)
- net NRF_RF: now also AE1.1 (FEED), L2.2
- net NRF_XC1: now also Y1.1, C17.1; no longer Y1.3
- net NRF_XC2: now also Y1.3, C18.1; no longer Y1.1
- new net: C12.2, D174.1 (K), L5.1, U2.7 (SW)
- new net: C15.2, R2.2, R3.1, U2.4 (FB)
- new net: R4.1, U2.3 (FREQ)
- new net: C12.1, U2.8 (BST)
- new net: C16.1, U2.1 (SS)
- new net: R1.1, U2.5 (EN)
- new net +3V3: C13.1, C14.1, C15.1, L5.2, R2.1, TP1.1
- new net V_EXT: C10.1, C11.1, J1.1 (Pin_1), R1.2, U2.6 (VIN)
Other:
- note added: "3V3 BUCK"
- note added: "ACDC Converter 48-24Vin"
- note removed: "Power"
- moved on the sheet: AE1, C1, C2, C3, C4, C5, C6, C7, C8, C9, D116, D117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

Commit message: layout progress
Parts:
- removed U1: NRF54L15-CAAA-Rx, ProjectFootprints:WLCSP 300, symbol ProjectSymbols:nRF54Lxx
- added C19, C20: 100n, Capacitor_SMD:C_0402_1005Metric, symbol Device:C_Small
- added J3: Conn_01x07_Pin, Connector_PinHeader_2.54mm:PinHeader_1x07_P2.54mm_Vertical, symbol Connector:Conn_01x07_Pin
- added U4: ~, ProjectFootprints:QFN-48_EP_6x6_Pitch0.4mm, symbol ProjectSymbols:nRF54L15-QFxx
- L5: LCSC (none) -> C2932476
Connections:
- net +3V3: now also J3.1 (Pin_1)
- net GND: now also C19.1, C20.1, J3.2 (Pin_2), U4.32 (VSS_PA), U4.44 (VSS), U4.49 (VSS)
- net LED_CIRCLE: now also J3.7 (Pin_7), U4.41 (P1.13)
- net LED_SEGMENTS: now also J3.6 (Pin_6), U4.42 (P1.14)
- net NRF_ANT: now also U4.31 (ANT)
- net NRF_NRST: now also J3.3 (Pin_3), U4.30 (nRESET)
- net NRF_SWDCLK: now also J3.4 (Pin_4), U4.26 (SWCLK)
- net NRF_SWDIO: now also J3.5 (Pin_5), U4.25 (SWDIO)
- net NRF_XC1: now also U4.34 (XC1)
- net NRF_XC2: now also U4.35 (XC2)
- net VDD_NRF: now also C19.2, C20.2, U4.10 (VDD), U4.22 (VDD), U4.36 (VDD), U4.47 (VDD), U4.48 (VDD)
- net at C5.2, C6.2, C7.2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: now also U4.33 (DECRF), U4.43 (DECA)
- net at C4.2, FB1.1, L1.2: now also U4.45 (DECD)
- net at L1.1: now also U4.46 (DCC)
Other:
- note added: "Connector"
- moved on the sheet: C1, C2, C3, J1

Commit message: finalized layout, everything on top + LCSC numbers
Parts:
- removed C10, C11: 4u7 100VDC, Capacitor_SMD:C_1206_3216Metric, symbol Device:C_Small
- removed C12: 100n 100VDC, Capacitor_SMD:C_0805_2012Metric, symbol Device:C_Small
- removed C13, C14: 22u 6.3V, Capacitor_SMD:C_0805_2012Metric, symbol Device:C_Small
- removed C15: 15p, Capacitor_SMD:C_0805_2012Metric, symbol Device:C_Small
- removed C16: 22n, Capacitor_SMD:C_0805_2012Metric, symbol Device:C_Small
- removed D174: ACDBMS2100-HF, Diode_SMD:D_SOD-123F, symbol Device:D_Schottky_Small_Filled
- removed L5: 10u, ProjectFootprints:NRS5040T3R3NMGJV, symbol Device:L_Small
- removed R1: 0R, Resistor_SMD:R_0805_2012Metric, symbol Device:R_Small
- removed R2: 210k, Resistor_SMD:R_0805_2012Metric, symbol Device:R_Small
- removed R3: 68k, Resistor_SMD:R_0805_2012Metric, symbol Device:R_Small
- removed R4: 47k, Resistor_SMD:R_0805_2012Metric, symbol Device:R_Small
- removed TP1, TP2: TestPoint, TestPoint:TestPoint_THTPad_2.0x2.0mm_Drill1.0mm, symbol Connector:TestPoint
- removed U2: MP4562, ProjectFootprints:MP4562, symbol ProjectSymbols:MP4562
- added C21: 100n, Capacitor_SMD:C_0402_1005Metric, symbol Device:C_Small
- added C22, C23: 47u 6.3V, Capacitor_SMD:C_0805_2012Metric, symbol Device:C_Small
- added C24, C25: 4u7 100VDC, Capacitor_SMD:C_1206_3216Metric, symbol Device:C_Small
- added C26: 10n, Capacitor_SMD:C_0402_1005Metric, symbol Device:C_Small
- added C27: ~, Capacitor_SMD:C_0603_1608Metric, symbol Device:C_Small
- added C28: 4n7, Capacitor_SMD:C_0603_1608Metric, symbol Device:C_Small
- added D175: B360, Diode_SMD:D_SMC, symbol Diode:B360
- added L6: 10u, ProjectFootprints:NRS5040T3R3NMGJV, symbol Device:L_Small
- added R10: 20k, Resistor_SMD:R_0805_2012Metric, symbol Device:R_Small
- added R11: 27k, Resistor_SMD:R_0805_2012Metric, symbol Device:R_Small
- added R12: 5.1k, Resistor_SMD:R_0402_1005Metric, symbol Device:R_Small
- added R5: 110k, Resistor_SMD:R_0805_2012Metric, symbol Device:R_Small
- added R7: 10k, Resistor_SMD:R_0402_1005Metric, symbol Device:R_Small
- added R9: 412k, Resistor_SMD:R_0805_2012Metric, symbol Device:R_Small
- added TP3, TP4: TestPoint, TestPoint:TestPoint_THTPad_2.0x2.0mm_Drill1.0mm, symbol Connector:TestPoint
- added U1: AMS1117-3.3, Package_TO_SOT_SMD:SOT-223-3_TabPin2, symbol Regulator_Linear:AMS1117-3.3
- added U3: TPS54260DGQ, Package_SO:MSOP-10-1EP_3x3mm_P0.5mm_EP2.2x3.1mm_Mask1.83x1.89mm_ThermalVias, symbol Regulator_Switching:TPS54260DGQ
- C19, C2, C20, C3: LCSC C1581 -> C696907
- U4: LCSC (none) -> C42458750
Connections:
- net VDD_NRF is gone; now on net +3V3: C1.2, C19.2, C2.2, C20.2, C3.2, U4.10 (VDD), U4.22 (VDD), U4.36 (VDD), U4.47 (VDD), U4.48 (VDD)
- net led_segment1/LED_BO is gone; now on net led_segment1/LED_DO: D116.4 (DI)
- net +3V3: now also U1.2 (VO)
- net +5V: now also C22.1, C23.1, L6.2, R11.1, TP3.1, U1.3 (VI)
- net GND: now also C22.2, C23.2, C24.2, C25.2, C26.2, C27.2, C28.2, D175.2 (A), R12.1, R7.1, R9.2, TP4.1, U1.1 (GND), U3.11 (EP), U3.9 (GND)
- net V_EXT: now also C24.1, C25.1, R5.1, U3.2 (VIN)
- net at D116.3 (DO), D117.4 (DI): now also D117.6 (BI)
- net at D116.1 (VCC): no longer D117.6 (BI)
- net led_segment2/LED_BI: no longer names the net of D117.1 (VCC)
- new net: R5.2, R7.2, U3.3 (EN)
- new net: R11.2, R12.2, U3.7 (VSENSE)
- new net: C27.1, R10.1, U3.8 (COMP)
- new net: C28.1, R10.2
- new net: C21.2, U3.1 (BOOT)
- new net: C21.1, D175.1 (K), L6.1, U3.10 (PH)
- new net: C26.1, U3.4 (SS/TR)
- new net: R9.1, U3.5 (RT/CLK)
- new net PWRGD: U3.6 (PWRGD)
- no-connect marks 5 -> 3
Other:
- sheet led_circle ports: added none; removed LED_BI, LED_BO
- sheet led_segment ports: added none; removed LED_BI, LED_BO
- sheet led_segment1 ports: added none; removed LED_BI, LED_BO
- sheet led_segment2 ports: added none; removed LED_BI, LED_BO
- sheet led_segment3 ports: added none; removed LED_BI, LED_BO
- note added: "5V Buck"
- note removed: "3V3 BUCK"
